File: pcb/pcb_REV2/rev2.brd (EAGLE design)
At the start: 94.8 x 88.1 mm, 70 parts, among them IC1 PIC24FJ128GA010, IC2 LM1117-XX, J1 RJ11-6X

Commit message: Schem
Parts:
- removed JP5: CELL (3.7V), pinhead:1X02
- added JP11, JP12: (no value), SparkFun:1X03
- added JP7: RPI SPI, pinhead:1X03
- added JP8: RPI PWR, pinhead:1X02
- added U$5: JST-PH_2-PIN_HEADER, SRG:JST_B2B-PH_HEADER
- JP1: value RPi -> gauge_selector; device pinhead:1X05 -> pinhead:1X03
- JP3: value SPDT -> main_power_switch
- moved JP1 203.6 mm to (-6.40, -148.1), turned to 0 degrees
- moved C3 7.30 mm to (78.8, 68.5), turned to 270 degrees
- moved C7 6.86 mm to (78.6, 75.1), turned to 270 degrees
- moved C11 4.33 mm to (78.5, 82.2)
- moved C12 2.24 mm to (83.3, 83.9), flipped to the bottom, turned to 0 degrees
- moved C10 2.22 mm to (83.4, 80.8)
- moved C8 2.16 mm to (83.4, 78.3)
- moved C4 1.70 mm to (83.7, 73.7), flipped to the bottom, turned to 270 degrees
- moved C1 1.29 mm to (84.6, 66.0)
- moved C2 0.91 mm to (84.5, 69.1)
Connections:
- removed net ADP_EN: U$3.P3
- new net ALT: JP12.1
- new net FG1_VCC: DSR2.2, DSR3.2, U$5.P1
- new net FG2_SCL: JP11.2
- new net FG2_SDA: JP11.1
- new net FG2_VCC: JP1.1, JP12.3
- net +5V: now also JP8.1; no longer JP1.1
- net 0V: no longer JP4.GND1, R11.1, R13.2
- net BATT+: now also U$3.P3; no longer DSR2.2, DSR3.2, JP5.2
- net BATT-: now also U$5.P2; no longer JP5.1
- net GND: now also JP11.3, JP12.2, JP4.GND1, JP8.2; no longer JP1.2
- net SCK1: now also JP7.3; no longer JP1.3
- net SDI1: now also JP7.2; no longer JP1.4
- net SDO1: now also JP7.1; no longer JP1.5
Routing:
- net N$8: track 42.3 -> 0.00 mm
- net N$9: track 40.6 -> 0.00 mm
- net GND: track 75.4 -> 116.0 mm, vias 7 -> 6
- net N$10: track 39.6 -> 0.00 mm
- net N$15: track 29.0 -> 0.00 mm
- net N$14: track 28.1 -> 0.00 mm
- net N$13: track 27.6 -> 0.00 mm
- net N$12: track 26.7 -> 0.00 mm
- net N$11: track 25.6 -> 0.14 mm
- net VDD: track 149.8 -> 167.6 mm
- net 0V: track 2.85 -> 18.9 mm
- net N$16: track 3.77 -> 12.1 mm
- net +5V: track 44.2 -> 37.2 mm
- net N$20: track 18.6 -> 13.4 mm, vias 1 -> 0
- net N$23: track 11.9 -> 6.85 mm, vias 1 -> 0
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