File: pcb/pcb_REV2/rev2.brd (EAGLE design)
At the start: 126.8 x 95.4 mm, 65 parts, among them IC1 PIC24FJ128GA010, IC2 LM1117-XX, IC3 MAX6520, J1 RJ11-6X

Commit message: version one done
Parts:
- moved ZD1 2.03 mm to (31.3, 31.5)
Routing:
- net N$36: track 0.00 -> 24.0 mm, vias 0 -> 2
- net N$37: track 7.54 -> 29.7 mm
- net VDD: track 44.5 -> 63.0 mm, vias 7 -> 8
- net N$39: track 0.00 -> 18.5 mm, vias 0 -> 2
- net +5V: track 30.5 -> 39.8 mm
- net N$31: track 0.00 -> 9.04 mm
- net BATT-: track 36.9 -> 42.3 mm
- net /MCLR: track 65.0 -> 67.2 mm

Commit message: go duck
Parts:
- added MAX_C1, MAX_C5: 150uF, adafruit:D/7343-31W
- added MAX_C2: 0.1u, eagle-ltspice:C1206
- added MAX_C6: 0.22u, eagle-ltspice:C1206
- added MAX_D: 200V 5A, diode:SMC
- added MAX_R2: 2, adafruit:R1206
- added U$3: MAX1708, max1708:QSOP16
- added U$6: (no value), fuelgauge:UP2B-2R2-R
Connections:
- new net N$30: MAX_C5.+
- new net N$35: MAX_D.A, U$3.3, U$3.4, U$3.5, U$6.P$2
- new net N$38: MAX_C2.1, MAX_R2.1, U$3.10, U$3.15, U$3.16
- new net N$40: MAX_C6.2, U$3.8
- new net VIN: MAX_C1.+, U$6.P$1
- new net VOUT: MAX_D.C, MAX_R2.2
- net GND: now also MAX_C1.-, MAX_C2.2, MAX_C5.-, MAX_C6.1, U$3.11, U$3.12, U$3.13, U$3.14, U$3.6, U$3.7, U$3.9
Changed lines of the file:
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@@
 <attribute name="OC_FARNELL" value="unknown" x="3.6576" y="32.1056" size="1.778" layer="27" display="off"/>
 </element>
+<element name="U$3" library="max1708" package="QSOP16" value="MAX1708" x="17.272" y="21.336" rot="R90"/>
+<element name="MAX_C1" library="adafruit" package="D/7343-31W" value="150uF" x="4.572" y="20.32" rot="R180"/>
+<element name="MAX_C5" library="adafruit" package="D/7343-31W" value="150uF" x="23.876" y="8.636" rot="R270"/>
+<element name="MAX_C6" library="eagle-ltspice" package="C1206" value="0.22u" x="59.944" y="17.272">
+<attribute name="SPICEMODEL" value="NONE" x="50.8" y="19.304" size="1.778" layer="27" display="off"/>
+<attribute name="SPICEPREFIX" value="C" x="50.8" y="19.304" size="1.778" layer="27" display="off"/>
+</element>
+<element name="MAX_D" library="diode" package="SMC" value="200V 5A" x="34.036" y="18.796" rot="R180"/>
+<element name="MAX_R2" library="adafruit" package="R1206" value="2" x="42.164" y="7.112"/>
+<element name="MAX_C2" library="eagle-ltspice" package="C1206" value="0.1u" x="55.372" y="10.16">
+<attribute name="SPICEMODEL" value="NONE" x="55.372" y="-10.16" size="1.778" layer="27" display="off"/>
+<attribute name="SPICEPREFIX" value="C" x="55.372" y="-10.16" size="1.778" layer="27" display="off"/>
+</element>
+<element name="U$6" library="fuelgauge" package="UP2B-2R2-R" value="" x="24.384" y="11.684"/>
 </elements>
 <signals>
@@
 <wire x1="5.872" y1="62.708" x2="6.096" y2="62.484" width="0.6096" layer="1"/>
 <wire x1="6.096" y1="62.484" x2="6.604" y2="62.484" width="0.6096" layer="1"/>
+<contactref element="U$3" pad="9"/>
+<contactref element="U$3" pad="11"/>
+<contactref element="U$3" pad="14"/>
+<contactref element="U$3" pad="13"/>
+<contactref element="U$3" pad="12"/>
+<contactref element="U$3" pad="6"/>
+<contactref element="MAX_C1" pad="-"/>
+<contactref element="MAX_C5" pad="-"/>
+<contactref element="MAX_C6" pad="1"/>
+<contactref element="U$3" pad="7"/>
+<contactref element="MAX_C2" pad="2"/>
+<wire x1="14.582" y1="22.2885" x2="14.582" y2="23.5585" width="0" layer="19" extent="1-1"/>
+<wire x1="19.962" y1="22.2885" x2="14.582" y2="22.2885" width="0" layer="19" extent="1-1"/>
 </signal>
 <signal name="VDD">
@@
 <wire x1="2.6808" y1="83.3628" x2="2.6808" y2="78.994" width="1.27" layer="1"/>
 <wire x1="2.6808" y1="78.994" x2="2.6808" y2="74.2696" width="1.27" layer="1"/>
-<wire x1="2.6808" y1="74.2696" x2="2.6808" y2="70.4712" width="1.27" layer="1"/>
-<wire x1="2.6808" y1="70.4712" x2="3.556" y2="69.596" width="1.27" layer="1"/>
-<wire x1="3.556" y1="69.596" x2="5.588" y2="69.596" width="0.6096" layer="1"/>
+<wire x1="3.4798" y1="69.596" x2="5.588" y2="69.596" width="0.6096" layer="1"/>
 <wire x1="5.588" y1="69.596" x2="6.096" y2="69.088" width="0.6096" layer="1"/>
 <wire x1="6.096" y1="69.088" x2="6.096" y2="65.308" width="0.6096" layer="1"/>
+<wire x1="3.4798" y1="69.596" x2="2.6924" y2="70.3834" width="0.6096" layer="1"/>
+<wire x1="2.6924" y1="70.3834" x2="2.6924" y2="74.258" width="0.6096" layer="1"/>
+<wire x1="2.6924" y1="74.258" x2="2.6808" y2="74.2696" width="0.6096" layer="1"/>
 </signal>
 <signal name="CS1">
@@
 <wire x1="54.864" y1="73.1516" x2="54.9144" y2="73.1012" width="0.6096" layer="1"/>
 </signal>
+<signal name="N$30">
+<contactref element="MAX_C5" pad="+"/>
+</signal>
+<signal name="N$35">
+<contactref element="MAX_D" pad="A"/>
+<contactref element="U$3" pad="4"/>
+<contactref element="U$3" pad="5"/>
+<contactref element="U$3" pad="3"/>
+<contactref element="U$6" pad="P$2"/>
+<wire x1="19.962" y1="20.3835" x2="30.336" y2="18.796" width="0" layer="19" extent="1-1"/>
+<wire x1="19.962" y1="21.0185" x2="19.962" y2="20.3835" width="0" layer="19" extent="1-1"/>
+<wire x1="19.962" y1="21.6535" x2="19.962" y2="21.0185" width="0" layer="19" extent="1-1"/>
+<wire x1="17.019" y1="12.684" x2="19.962" y2="20.3835" width="0" layer="19" extent="1-1"/>
+</signal>
+<signal name="N$38">
+<contactref element="U$3" pad="16"/>
+<contactref element="U$3" pad="10"/>
+<contactref element="U$3" pad="15"/>
+<contactref element="MAX_R2" pad="1"/>
+<contactref element="MAX_C2" pad="1"/>
+<wire x1="40.742" y1="7.112" x2="53.972" y2="10.16" width="0" layer="19" extent="1-1"/>
+<wire x1="14.582" y1="19.1135" x2="40.742" y2="7.112" width="0" layer="19" extent="1-1"/>
+<wire x1="14.582" y1="19.7485" x2="14.582" y2="19.1135" width="0" layer="19" extent="1-1"/>
+<wire x1="14.582" y1="22.9235" x2="14.582" y2="19.7485" width="0" layer="19" extent="1-1"/>
+</signal>
+<signal name="VOUT">
+<contactref element="MAX_D" pad="C"/>
+<contactref element="MAX_R2" pad="2"/>
+<wire x1="43.586" y1="7.112" x2="37.736" y2="18.796" width="0" layer="19" extent="1-1"/>
+</signal>
+<signal name="VIN">
+<contactref element="MAX_C1" pad="+"/>
+<contactref element="U$6" pad="P$1"/>
+<wire x1="5.114" y1="12.684" x2="1.197" y2="20.32" width="0" layer="19" extent="1-1"/>
+</signal>
+<signal name="N$40">
+<contactref element="U$3" pad="8"/>
+<contactref element="MAX_C6" pad="2"/>
+<wire x1="19.962" y1="23.5585" x2="61.344" y2="17.272" width="0" layer="19" extent="1-1"/>
+</signal>
+<signal name="N$41">
+<via x="6.8834" y="65.278" extent="1-16" drill="0.6"/>
+</signal>
+<signal name="N$42">
+<via x="17.018" y="65.3034" extent="1-16" drill="0.6"/>
+</signal>
+<signal name="N$43">
+<via x="18.5166" y="65.3288" extent="1-16" drill="0.6"/>
+</signal>
+<signal name="N$44">
+<via x="19.685" y="64.6684" extent="1-16" drill="0.6"/>
+</signal>
+<signal name="N$45">
+<via x="20.7264" y="63.5508" extent="1-16" drill="0.6"/>
+</signal>
 </signals>

Commit message: VERSION 1 with everything
Parts:
- removed MAX_C6: 0.22u, eagle-ltspice:C1206
- added MAX_C4: 0.22u, eagle-ltspice:C1206
- MAX_C2: value 0.1u -> 150uF; device eagle-ltspice:C1206 -> adafruit:D/7343-31W
- MAX_C5: value 150uF -> 0.1u; device adafruit:D/7343-31W -> eagle-ltspice:C1206
- U$6: device fuelgauge:UP2B-2R2-R -> duckgauge:UP2B-2R2-R
- moved MAX_C2 37.6 mm to (20.8, 24.9)
- moved MAX_C5 27.7 mm to (48.3, 21.8), turned to 90 degrees
- moved U$3 21.9 mm to (39.1, 20.3), turned to 0 degrees
- moved U$6 18.9 mm to (7.11, 4.06), turned to 270 degrees
- moved MAX_C1 16.4 mm to (20.8, 18.3)
- moved MAX_R2 14.9 mm to (44.7, 21.8), turned to 90 degrees
- moved MAX_D 3.87 mm to (30.5, 20.3), turned to 270 degrees
- moved RSNS 3.05 mm to (20.9, 33.2)
- moved U$1 2.54 mm to (21.1, 29.9)
Connections:
- removed net N$30: MAX_C5.+
- removed net VIN: MAX_C1.+, U$6.P$1
- removed net VOUT: MAX_D.C, MAX_R2.2
- net +5V: now also MAX_C2.+, MAX_D.C, MAX_R2.2
- net AVIN: now also MAX_C1.+, U$6.P$1
- net GND: now also MAX_C2.-, MAX_C4.1, MAX_C5.2; no longer MAX_C2.2, MAX_C5.-, MAX_C6.1
- net N$38: now also MAX_C5.1; no longer MAX_C2.1
- net N$40: now also MAX_C4.2; no longer MAX_C6.2
Routing:
- net AVIN: track 16.7 -> 72.3 mm, vias 0 -> 2
- net N$35: track 0.00 -> 41.1 mm
- net +5V: track 39.8 -> 71.9 mm
- net GND: track 79.7 -> 102.4 mm
- net N$40: track 0.00 -> 17.5 mm, vias 0 -> 2
- net N$38: track 0.00 -> 16.7 mm
- net N$36: track 24.0 -> 20.4 mm
- net N$37: track 29.7 -> 26.2 mm, vias 0 -> 2
- net PIO: track 50.7 -> 53.2 mm
- net N$39: track 18.5 -> 20.3 mm
- net N$31: track 9.04 -> 10.1 mm
- added copper zone on layer 1, net AVIN

Commit message: VERSION UNRELIABLE
Parts:
- removed JP4: USB_MICROB_PLUGCONN-11752, SparkFun-Connectors:USB-B-MICRO-SMD_V03
- added U$7: MICRO-USB-SHIELD-ZX62R-B-5P, con-hirose:ZX62R-B-5P
- LED1, LED2, LED3: value LAP4-BOTTOM -> (none); device led:P47F-BOTTOM -> led:1206
- moved C10 8.23 mm to (83.3, 70.1)
- moved C11 8.23 mm to (83.3, 73.0)
- moved C12 8.23 mm to (83.3, 76.0)
- moved C15 8.23 mm to (36.8, 29.2)
- moved C16 8.23 mm to (63.8, 51.9)
- moved C17 8.23 mm to (60.2, 76.6)
- moved C2 8.23 mm to (83.4, 59.2)
- moved C27 8.23 mm to (65.1, 56.4)
- moved C3 8.23 mm to (83.4, 62.1)
- moved C4 8.23 mm to (83.4, 65.0)
- moved C6 8.23 mm to (58.8, 57.7)
- moved C7 8.23 mm to (83.3, 64.0)
- moved C8 8.23 mm to (83.3, 67.2)
- moved DSR3 8.23 mm to (7.11, 33.1)
- moved IC2 8.23 mm to (32.2, 47.3)
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Connections:
- net GND: now also U$7.1, U$7.M1, U$7.M2, U$7.M3, U$7.M4; no longer JP4.GND1
- net VDDUSB: now also U$7.5; no longer JP4.VBUS1
Routing:
- net AVIN: track 72.3 -> 85.5 mm
- net GND: track 102.4 -> 96.5 mm
- net VDDUSB: track 31.5 -> 32.6 mm
- net N$3: track 4.21 -> 5.23 mm
- net N$18: track 4.26 -> 5.28 mm
- net N$32: track 4.28 -> 5.31 mm
- removed copper zone on layer 1, net AVIN
Other:
- board size 126.8 x 95.4 mm -> 95.2 x 80 mm
- board text added: "ECE477 TEAM7 SPRING 2015"
- board text added: "VERSION UNRELIABLE"

Commit message: latest
Parts:
- removed C20, C21: 0.1uF, rcl:C1206
- removed DSR1: 150, rcl:R1206
- removed DSR2: 500, rcl:R1206
- removed DSR3: 1K, rcl:R1206
- removed IC3: MAX6520, maxim:SOT23
- removed JP1: gauge_selector, pinhead:1X03
- removed RSNS: (no value), rcl:R1206
- removed U$1: DS2781E, fuelgauge:TSSOP8
- removed U$5: JST-PH_2-PIN_HEADER, SRG:JST_B2B-PH_HEADER
- removed ZD1: 5.6V, diode:SOD80C
- MAX_C1, MAX_C2: device adafruit:D/7343-31W -> rcl:CT7343
- moved R8 28.4 mm to (28.3, 51.1), turned to 270 degrees
- moved LED1 28.2 mm to (28.3, 59.2), turned to 270 degrees
- moved MAX_C4 24.4 mm to (11.4, 5.84)
- moved R7 22.4 mm to (24.0, 51.1), turned to 270 degrees
- moved MAX_R2 22.1 mm to (25.2, 3.15), turned to 0 degrees
- moved LED2 22.1 mm to (24.0, 59.2), turned to 270 degrees
- moved MAX_C5 20.6 mm to (29.2, 5.99), turned to 0 degrees
- moved C15 18.4 mm to (37.9, 10.8), turned to 270 degrees
- moved U$3 18.3 mm to (21.2, 8.13), turned to 270 degrees
- moved LMC2 17.5 mm to (29.4, 36.9), turned to 0 degrees
- moved JP12 17.2 mm to (7.06, 43.0), turned to 270 degrees
- moved JP6 16.6 mm to (37.5, 37.8), turned to 0 degrees
- moved R9 16.2 mm to (19.3, 51.0), turned to 90 degrees
- moved JP11 16.0 mm to (48.9, 9.60)
- moved JP8 16.0 mm to (41.2, 4.88)
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Connections:
- removed net BATT-: C20.2, C21.2, IC3.3, RSNS.2, U$1.2, U$5.P2
- removed net FG2_VCC: JP1.1, JP12.3
- removed net N$31: DSR1.2, U$1.5, ZD1.C
- removed net N$36: C21.1, DSR2.1, U$1.4
- removed net N$37: C20.1, U$1.1, U$1.6
- removed net N$39: DSR3.1, U$1.3
- removed net REAL_BATT+: DSR2.2, DSR3.2, JP1.3, U$5.P1
- net BATT+: now also JP12.3; no longer JP1.2
- net DS_DATA: no longer DSR1.1
- net GND: no longer IC3.1, IC3.2, RSNS.1, U$1.7, ZD1.A
- net PIO: no longer U$1.8
Routing:
- net PIO: track 53.2 -> 0.00 mm, vias 2 -> 0
- net DS_DATA: track 42.5 -> 0.00 mm
- net BATT-: track 41.9 -> 0.00 mm
- net AVIN: track 85.5 -> 50.6 mm, vias 2 -> 0
- net REAL_BATT+: track 26.3 -> 0.00 mm
- net N$37: track 26.2 -> 0.00 mm, vias 2 -> 0
- net N$36: track 20.4 -> 0.00 mm, vias 2 -> 0
- net N$39: track 20.3 -> 0.00 mm, vias 2 -> 0
- net N$35: track 41.1 -> 25.6 mm
- net N$40: track 17.5 -> 5.79 mm, vias 2 -> 0
- net N$31: track 10.1 -> 0.00 mm
- net N$51: track 21.3 -> 11.7 mm
- net FG2_VCC: track 7.70 -> 0.00 mm
- net N$38: track 16.7 -> 23.9 mm
- net GND: track 96.5 -> 101.3 mm, vias 9 -> 11
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Other:
- board size 95.2 x 80 mm -> 95.2 x 64.3 mm
- board text added: "VERSION KIND OF GOOD"
- board text removed: "VERSION UNRELIABLE"
