File: pcb/pcb_REV2/rev2.sch (EAGLE design)
At the start: 70 parts, among them IC1 PIC24FJ128GA010, IC2 LM1117-XX, J1 RJ11-6X

Commit message: Schem
Parts:
- removed JP5: CELL (3.7V), pinhead:PINHD-1X2
- added JP11, JP12: (no value), SparkFun:M03PTH
- added JP7: RPI SPI, pinhead:PINHD-1X3
- added JP8: RPI PWR, pinhead:PINHD-1X2
- added U$5: JST-PH_2-PIN_HEADER, SRG:JST-PH_2-PIN_HEADER
- JP1: value RPi -> gauge_selector; device pinhead:PINHD-1X5 -> pinhead:PINHD-1X3
- JP3: value SPDT -> main_power_switch
Connections:
- removed net ADP_EN: U$3.EN
- new net ALT: JP12.1
- new net FG1_VCC: DSR2.2, DSR3.2, U$5.1
- new net FG2_SCL: JP11.2
- new net FG2_SDA: JP11.1
- new net FG2_VCC: JP1.1, JP12.3
- net +5V: now also JP8.1; no longer JP1.1
- net 0V: no longer JP4.GND, R11.1, R13.2
- net BATT+: now also U$3.EN; no longer DSR2.2, DSR3.2, JP5.2
- net BATT-: now also U$5.2; no longer JP5.1
- net GND: now also JP11.3, JP12.2, JP4.GND, JP8.2; no longer JP1.2
- net SCK1: now also JP7.3; no longer JP1.3
- net SDI1: now also JP7.2; no longer JP1.4
- net SDO1: now also JP7.1; no longer JP1.5
Other:
- note added: "gauge selector is a Switch that chooses between Fuel Gauge A and Fuel Gauge B (Which sid just found at 4AM). We can choose which one to use by flipping the switch."

Commit message: Kenzhebalin
Parts:
- removed ACCOMP, ACIN, CSS: .1u, rcl:C-EUC1206
- removed AR1, ARCOMP: 4.7K, rcl:R-US_M2012
- removed AR2: 12.4k, rcl:R-US_M2012
- removed AZD1: DIODE-ZENERSMB, SparkFun-DiscreteSemi:DIODE-ZENERSMB
- removed L1: (no value), inductor-neosid:SM-NE45
- removed R6: NL, rcl:R-US_M2012
- removed U$3: ADP1613, adp1613:ADP1613
- added IC3: MAX6520, maxim:MAX6520
- DSR1, DSR2, DSR3, R1, R11, R2, R3, R4, R5, R7, R8, R9, RSNS: device rcl:R-US_M2012 -> rcl:R-US_R1206
- Q1: device crystal:CRYTALHC49UP -> crystal:CRYTALHC49U-V
Connections:
- removed net 0V: C37.1, C38.1, U$2.VSS
- removed net ADP_FREQ: U$3.FREQ
- removed net FG1_VCC: DSR2.2, DSR3.2, U$5.1
- removed net N$30: CSS.1, U$3.SS
- removed net N$38: AZD1.A, L1.1, U$3.SW
- removed net N$40: ACCOMP.1, ARCOMP.1
- removed net N$41: AR1.1, AR2.1, U$3.FB
- removed net N$42: ARCOMP.2, U$3.COMP
- removed net N$50: IC1.!MCLR, R3.1
- new net N$4: IC1.!MCLR, R3.1, R5.1
- new net REAL_BATT+: DSR2.2, DSR3.2, JP1.3, U$5.1
- net +5V: no longer AR1.2, AZD1.C
- net /MCLR: no longer R5.1
- net AVIN: now also IC2.IN, LMC1.1; no longer ACIN.1, L1.2, U$3.VIN
- net BATT+: now also JP1.2; no longer IC2.IN, LMC1.1, U$3.EN
- net BATT-: now also IC3.GND
- net DS_DATA: now also IC1.U1RX/RF2; no longer IC1.PGD1/EMUD1/AN0/CN2/RB0
- net FG2_SCL: now also IC1.SCL2/RA2
- net FG2_SDA: now also IC1.SDA2/RA3
- net GND: now also C37.1, C38.1, IC3.IN, IC3.OUT, R11.1, R13.2, U$2.VSS; no longer ACCOMP.2, ACIN.2, AR2.2, CSS.2, U$3.GND
- net OSC1: no longer R6.1
- net PIO: now also IC1.U1TX/RF3; no longer IC1.PGC1/EMUC1/AN1/CN3/RB1
- net VDD: no longer R6.2
Other:
- moved on the sheet: C20, DSR2, DSR3, R3, U$1

Commit message: go duck
Parts:
- added MAX_C1, MAX_C5: 150uF, adafruit:CPOL-USD/7343-31W
- added MAX_C2: 0.1u, eagle-ltspice:CC1206
- added MAX_C6: 0.22u, eagle-ltspice:CC1206
- added MAX_D: 200V 5A, diode:SCHOTTKY-DIODESMC
- added MAX_R2: 2, adafruit:R-US_R1206
- added U$3: MAX1708, max1708:MAX1708
- added U$6: (no value), fuelgauge:UP2B-2R2-R
Connections:
- new net N$30: MAX_C5.+
- new net N$35: MAX_D.A, U$3.3_LX, U$3.4_LX, U$3.5_LX, U$6.P$2
- new net N$38: MAX_C2.1, MAX_R2.1, U$3.10_OUT, U$3.15_3.3/5, U$3.16_CLK
- new net N$40: MAX_C6.2, U$3.8_REF
- new net VIN: MAX_C1.+, U$6.P$1
- new net VOUT: MAX_D.C, MAX_R2.2
- net GND: now also MAX_C1.-, MAX_C2.2, MAX_C5.-, MAX_C6.1, U$3.11_FB, U$3.12_PGND, U$3.13_PGND, U$3.14_PGND, U$3.6_GND, U$3.7_SS/LIM, U$3.9_GND
Other:
- moved on the sheet: IC2, JP1, JP11, JP12, LMC1, LMC2

Commit message: VERSION 1 with everything
Parts:
- MAX_C2: value 0.1u -> 150uF; device eagle-ltspice:CC1206 -> adafruit:CPOL-USD/7343-31W
- MAX_C5: value 150uF -> 0.1u; device adafruit:CPOL-USD/7343-31W -> eagle-ltspice:CC1206
- U$6: device fuelgauge:UP2B-2R2-R -> duckgauge:UP2B-2R2-R
- renumbered MAX_C6 to MAX_C4
Connections:
- removed net N$30: MAX_C5.+
- removed net VIN: MAX_C1.+, U$6.P$1
- removed net VOUT: MAX_D.C, MAX_R2.2
- net +5V: now also MAX_C2.+, MAX_D.C, MAX_R2.2
- net AVIN: now also MAX_C1.+, U$6.P$1
- net GND: now also MAX_C2.-, MAX_C5.2; no longer MAX_C2.2, MAX_C5.-
- net N$38: now also MAX_C5.1; no longer MAX_C2.1
Other:
- moved on the sheet: MAX_D
Changed lines of the file:
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@@
 <part name="U$3" library="max1708" deviceset="MAX1708" device=""/>
 <part name="MAX_C1" library="adafruit" deviceset="CPOL-US" device="D/7343-31W" value="150uF"/>
-<part name="MAX_C5" library="adafruit" deviceset="CPOL-US" device="D/7343-31W" value="150uF"/>
-<part name="MAX_C6" library="eagle-ltspice" deviceset="C" device="C1206" value="0.22u"/>
+<part name="MAX_C2" library="adafruit" deviceset="CPOL-US" device="D/7343-31W" value="150uF"/>
+<part name="MAX_C4" library="eagle-ltspice" deviceset="C" device="C1206" value="0.22u"/>
 <part name="MAX_D" library="diode" deviceset="SCHOTTKY-DIODE" device="SMC" value="200V 5A"/>
 <part name="MAX_R2" library="adafruit" deviceset="R-US_" device="R1206" value="2"/>
-<part name="MAX_C2" library="eagle-ltspice" deviceset="C" device="C1206" value="0.1u"/>
-<part name="U$6" library="fuelgauge" deviceset="UP2B-2R2-R" device=""/>
+<part name="MAX_C5" library="eagle-ltspice" deviceset="C" device="C1206" value="0.1u"/>
+<part name="U$6" library="duckgauge" deviceset="UP2B-2R2-R" device=""/>
 </parts>
 <sheets>
@@
 <instance part="U$3" gate="G$1" x="27.94" y="55.88"/>
 <instance part="MAX_C1" gate="G$1" x="15.24" y="91.44"/>
-<instance part="MAX_C5" gate="G$1" x="76.2" y="93.98"/>
-<instance part="MAX_C6" gate="G$1" x="17.78" y="63.5" rot="R90"/>
-<instance part="MAX_D" gate="G$1" x="50.8" y="101.6"/>
+<instance part="MAX_C2" gate="G$1" x="76.2" y="91.44"/>
+<instance part="MAX_C4" gate="G$1" x="17.78" y="63.5" rot="R90"/>
+<instance part="MAX_D" gate="G$1" x="53.34" y="101.6"/>
 <instance part="MAX_R2" gate="G$1" x="63.5" y="91.44" rot="R90"/>
-<instance part="MAX_C2" gate="G$1" x="66.04" y="71.12" rot="R90"/>
+<instance part="MAX_C5" gate="G$1" x="66.04" y="71.12" rot="R90"/>
 <instance part="U$6" gate="G$1" x="15.24" y="119.38" rot="R90"/>
 </instances>
@@
 <wire x1="63.5" y1="50.8" x2="76.2" y2="50.8" width="0.1524" layer="91"/>
 <wire x1="76.2" y1="50.8" x2="76.2" y2="81.28" width="0.1524" layer="91"/>
-<wire x1="76.2" y1="81.28" x2="76.2" y2="88.9" width="0.1524" layer="91"/>
+<wire x1="76.2" y1="81.28" x2="76.2" y2="86.36" width="0.1524" layer="91"/>
 <wire x1="76.2" y1="81.28" x2="86.36" y2="81.28" width="0.1524" layer="91"/>
 <label x="83.82" y="81.28" size="1.778" layer="95"/>
@@
 <label x="7.62" y="88.9" size="1.778" layer="95" rot="R90"/>
 <pinref part="MAX_C1" gate="G$1" pin="-"/>
-<pinref part="MAX_C5" gate="G$1" pin="-"/>
-<pinref part="MAX_C6" gate="G$1" pin="1"/>
+<pinref part="MAX_C2" gate="G$1" pin="-"/>
+<pinref part="MAX_C4" gate="G$1" pin="1"/>
 <pinref part="U$3" gate="G$1" pin="7_SS/LIM"/>
 <wire x1="12.7" y1="68.58" x2="22.86" y2="68.58" width="0.1524" layer="91"/>
-<pinref part="MAX_C2" gate="G$1" pin="2"/>
+<pinref part="MAX_C5" gate="G$1" pin="2"/>
+<junction x="63.5" y="66.04"/>
+<junction x="12.7" y="63.5"/>
 </segment>
 </net>
@@
 <junction x="256.286" y="88.9"/>
 <pinref part="JP8" gate="G$1" pin="1"/>
+</segment>
+<segment>
+<wire x1="81.28" y1="101.6" x2="76.2" y2="101.6" width="0.1524" layer="91"/>
+<wire x1="76.2" y1="101.6" x2="63.5" y2="101.6" width="0.1524" layer="91"/>
+<wire x1="63.5" y1="101.6" x2="63.5" y2="96.52" width="0.1524" layer="91"/>
+<wire x1="63.5" y1="101.6" x2="55.88" y2="101.6" width="0.1524" layer="91"/>
+<label x="83.82" y="101.6" size="1.778" layer="95" rot="R90"/>
+<pinref part="MAX_D" gate="G$1" pin="C"/>
+<pinref part="MAX_R2" gate="G$1" pin="2"/>
+<wire x1="76.2" y1="93.98" x2="76.2" y2="101.6" width="0.1524" layer="91"/>
+<pinref part="MAX_C2" gate="G$1" pin="+"/>
+<junction x="76.2" y="101.6"/>
+<junction x="63.5" y="101.6"/>
 </segment>
 </net>
@@
 <junction x="170.18" y="55.88"/>
 </segment>
+<segment>
+<wire x1="15.24" y1="93.98" x2="15.24" y2="101.6" width="0.1524" layer="91"/>
+<wire x1="10.16" y1="101.6" x2="7.62" y2="101.6" width="0.1524" layer="91"/>
+<label x="10.16" y="101.6" size="1.778" layer="95" rot="R90"/>
+<pinref part="MAX_C1" gate="G$1" pin="+"/>
+<pinref part="U$6" gate="G$1" pin="P$1"/>
+<wire x1="15.24" y1="101.6" x2="10.16" y2="101.6" width="0.1524" layer="91"/>
+<junction x="10.16" y="101.6"/>
+</segment>
 </net>
 <net name="FG2_VCC" class="0">
@@
 </segment>
 </net>
-<net name="N$30" class="0">
-<segment>
-<wire x1="76.2" y1="96.52" x2="76.2" y2="101.6" width="0.1524" layer="91"/>
-<pinref part="MAX_C5" gate="G$1" pin="+"/>
-</segment>
-</net>
 <net name="N$35" class="0">
 <segment>
-<wire x1="48.26" y1="101.6" x2="45.72" y2="101.6" width="0.1524" layer="91"/>
+<wire x1="50.8" y1="101.6" x2="45.72" y2="101.6" width="0.1524" layer="91"/>
 <wire x1="45.72" y1="101.6" x2="40.64" y2="101.6" width="0.1524" layer="91"/>
 <wire x1="40.64" y1="96.52" x2="40.64" y2="101.6" width="0.1524" layer="91"/>
@@
 <junction x="63.5" y="76.2"/>
 <pinref part="MAX_R2" gate="G$1" pin="1"/>
-<pinref part="MAX_C2" gate="G$1" pin="1"/>
+<pinref part="MAX_C5" gate="G$1" pin="1"/>
 <junction x="63.5" y="71.12"/>
 </segment>
 </net>
-<net name="VOUT" class="0">
-<segment>
-<wire x1="81.28" y1="101.6" x2="63.5" y2="101.6" width="0.1524" layer="91"/>
-<wire x1="63.5" y1="101.6" x2="63.5" y2="96.52" width="0.1524" layer="91"/>
-<wire x1="63.5" y1="101.6" x2="53.34" y2="101.6" width="0.1524" layer="91"/>
-<label x="83.82" y="101.6" size="1.778" layer="95" rot="R90"/>
-<pinref part="MAX_D" gate="G$1" pin="C"/>
-<pinref part="MAX_R2" gate="G$1" pin="2"/>
-</segment>
-</net>
-<net name="VIN" class="0">
-<segment>
-<wire x1="15.24" y1="93.98" x2="15.24" y2="101.6" width="0.1524" layer="91"/>
-<wire x1="10.16" y1="101.6" x2="7.62" y2="101.6" width="0.1524" layer="91"/>
-<label x="10.16" y="101.6" size="1.778" layer="95" rot="R90"/>
-<pinref part="MAX_C1" gate="G$1" pin="+"/>
-<pinref part="U$6" gate="G$1" pin="P$1"/>
-<wire x1="15.24" y1="101.6" x2="10.16" y2="101.6" width="0.1524" layer="91"/>
-<junction x="10.16" y="101.6"/>
-</segment>
-</net>
 <net name="N$40" class="0">
 <segment>
 <pinref part="U$3" gate="G$1" pin="8_REF"/>
-<pinref part="MAX_C6" gate="G$1" pin="2"/>
-</segment>
-</net>
+<pinref part="MAX_C4" gate="G$1" pin="2"/>
+</segment>
+</net>

Commit message: VERSION UNRELIABLE
Parts:
- removed JP4: USB_MICROB_PLUGCONN-11752, SparkFun-Connectors:USB_MICROB_PLUGCONN-11752
- added U$7: MICRO-USB-SHIELD-ZX62R-B-5P, con-hirose:MICRO-USB-SHIELD-ZX62R-B-5P
- LED1, LED2, LED3: value LAP4-BOTTOM -> (none); device led:LAP4-BOTTOM -> led:LEDSMT1206
Connections:
- net GND: now also U$7G$1.S1, U$7G$1.S2, U$7G$1.S3, U$7G$1.S4, U$7G$2.1; no longer JP4.GND
- net VDDUSB: now also U$7G$2.5; no longer JP4.VCC
Other:
- moved on the sheet: C37
Changed lines of the file:
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@@
 <part name="SUPPLY42" library="supply2" deviceset="GND" device=""/>
 <part name="U$2" library="fuelgauge" deviceset="MCP73833" device=""/>
-<part name="JP4" library="SparkFun-Connectors" deviceset="USB_MICROB_PLUG" device="CONN-11752"/>
 <part name="C37" library="rcl" deviceset="C-EU" device="C1206" value=".1u"/>
 <part name="R7" library="rcl" deviceset="R-US_" device="R1206" value="100"/>
 <part name="R8" library="rcl" deviceset="R-US_" device="R1206" value="100"/>
 <part name="R9" library="rcl" deviceset="R-US_" device="R1206" value="100"/>
-<part name="LED1" library="led" deviceset="*P4" device="-BOTTOM" technology="LA"/>
-<part name="LED2" library="led" deviceset="*P4" device="-BOTTOM" technology="LA"/>
-<part name="LED3" library="led" deviceset="*P4" device="-BOTTOM" technology="LA"/>
+<part name="LED1" library="led" deviceset="LED" device="SMT1206"/>
+<part name="LED2" library="led" deviceset="LED" device="SMT1206"/>
+<part name="LED3" library="led" deviceset="LED" device="SMT1206"/>
 <part name="R11" library="rcl" deviceset="R-US_" device="R1206" value="100"/>
 <part name="R13" library="varistor" deviceset="THERMISTOR" device="-5"/>
@@
 <part name="MAX_C5" library="eagle-ltspice" deviceset="C" device="C1206" value="0.1u"/>
 <part name="U$6" library="duckgauge" deviceset="UP2B-2R2-R" device=""/>
+<part name="U$7" library="con-hirose" deviceset="MICRO-USB-SHIELD-" device="ZX62R-B-5P"/>
+<part name="OUTPUT2" library="supply2" deviceset="GND" device=""/>
 </parts>
 <sheets>
@@
 <instance part="SUPPLY42" gate="GND" x="269.24" y="167.64" rot="R180"/>
 <instance part="U$2" gate="G$1" x="38.1" y="187.96"/>
-<instance part="JP4" gate="G$1" x="12.7" y="198.12" rot="R180"/>
-<instance part="C37" gate="G$1" x="30.48" y="198.12"/>
+<instance part="C37" gate="G$1" x="40.64" y="200.66" rot="R270"/>
 <instance part="R7" gate="G$1" x="17.78" y="182.88"/>
 <instance part="R8" gate="G$1" x="12.7" y="185.42"/>
@@
 <instance part="SUPPLY35" gate="GND" x="60.96" y="165.1"/>
 <instance part="SUPPLY36" gate="GND" x="71.12" y="165.1"/>
-<instance part="OUTPUT37" gate="GND" x="24.892" y="200.66"/>
+<instance part="OUTPUT37" gate="GND" x="12.7" y="195.58"/>
 <instance part="IC3" gate="-1" x="53.34" y="10.16" rot="R180"/>
-<instance part="SUPPLY38" gate="GND" x="35.56" y="198.12"/>
+<instance part="SUPPLY38" gate="GND" x="43.18" y="198.12"/>
 <instance part="SUPPLY39" gate="GND" x="20.32" y="177.8"/>
 <instance part="SUPPLY40" gate="GND" x="55.88" y="198.12"/>
@@
 <instance part="MAX_C5" gate="G$1" x="66.04" y="71.12" rot="R90"/>
 <instance part="U$6" gate="G$1" x="15.24" y="119.38" rot="R90"/>
+<instance part="U$7" gate="G$1" x="27.94" y="208.28" rot="R90"/>
+<instance part="U$7" gate="G$2" x="17.78" y="203.2" rot="R90"/>
+<instance part="OUTPUT2" gate="GND" x="35.56" y="208.28" rot="R90"/>
 </instances>
 <busses>
@@
 </segment>
 <segment>
-<pinref part="JP4" gate="G$1" pin="GND"/>
-<wire x1="20.32" y1="203.2" x2="24.892" y2="203.2" width="0.1524" layer="91"/>
-<pinref part="OUTPUT37" gate="GND" pin="GND"/>
-</segment>
-<segment>
 <pinref part="R13" gate="G$1" pin="2"/>
 <pinref part="SUPPLY36" gate="GND" pin="GND"/>
@@
 <segment>
 <pinref part="C37" gate="G$1" pin="1"/>
-<wire x1="35.56" y1="200.66" x2="30.48" y2="200.66" width="0.1524" layer="91"/>
 <pinref part="SUPPLY38" gate="GND" pin="GND"/>
 </segment>
@@
 <junction x="12.7" y="63.5"/>
 </segment>
+<segment>
+<pinref part="U$7" gate="G$1" pin="S1"/>
+<pinref part="U$7" gate="G$1" pin="S2"/>
+<wire x1="30.48" y1="200.66" x2="30.48" y2="203.2" width="0.1524" layer="91"/>
+<pinref part="U$7" gate="G$1" pin="S3"/>
+<wire x1="30.48" y1="203.2" x2="30.48" y2="205.74" width="0.1524" layer="91"/>
+<pinref part="U$7" gate="G$1" pin="S4"/>
+<wire x1="30.48" y1="205.74" x2="30.48" y2="208.28" width="0.1524" layer="91"/>
+<wire x1="30.48" y1="208.28" x2="33.02" y2="208.28" width="0.1524" layer="91"/>
+<pinref part="OUTPUT2" gate="GND" pin="GND"/>
+</segment>
+<segment>
+<pinref part="U$7" gate="G$2" pin="1"/>
+<pinref part="OUTPUT37" gate="GND" pin="GND"/>
+</segment>
 </net>
 <net name="N$1" class="0">
@@
 <wire x1="7.62" y1="167.64" x2="5.08" y2="167.64" width="0.1524" layer="91"/>
 <wire x1="5.08" y1="167.64" x2="5.08" y2="187.96" width="0.1524" layer="91"/>
-<pinref part="JP4" gate="G$1" pin="VCC"/>
-<wire x1="20.32" y1="193.04" x2="22.86" y2="193.04" width="0.1524" layer="91"/>
-<wire x1="22.86" y1="193.04" x2="27.94" y2="193.04" width="0.1524" layer="91"/>
-<wire x1="22.86" y1="193.04" x2="22.86" y2="190.5" width="0.1524" layer="91"/>
+<wire x1="22.86" y1="195.58" x2="22.86" y2="190.5" width="0.1524" layer="91"/>
 <pinref part="U$2" gate="G$1" pin="VDD@1"/>
 <wire x1="22.86" y1="190.5" x2="27.94" y2="190.5" width="0.1524" layer="91"/>
@@
 <wire x1="20.32" y1="187.96" x2="20.32" y2="190.5" width="0.1524" layer="91"/>
 <wire x1="20.32" y1="190.5" x2="22.86" y2="190.5" width="0.1524" layer="91"/>
-<wire x1="27.94" y1="193.04" x2="27.94" y2="203.2" width="0.1524" layer="91"/>
+<wire x1="33.02" y1="200.66" x2="33.02" y2="203.2" width="0.1524" layer="91"/>
 <pinref part="LED3" gate="G$1" pin="A"/>
-<wire x1="27.94" y1="203.2" x2="55.88" y2="203.2" width="0.1524" layer="91"/>
-<junction x="22.86" y="193.04"/>
+<wire x1="33.02" y1="203.2" x2="55.88" y2="203.2" width="0.1524" layer="91"/>
 <junction x="7.62" y="167.64"/>
 <pinref part="C37" gate="G$1" pin="2"/>
-<wire x1="30.48" y1="193.04" x2="27.94" y2="193.04" width="0.1524" layer="91"/>
-<junction x="27.94" y="193.04"/>
-</segment>
-</net>
+<wire x1="35.56" y1="200.66" x2="33.02" y2="200.66" width="0.1524" layer="91"/>
+<junction x="33.02" y="200.66"/>
+<wire x1="22.86" y1="195.58" x2="33.02" y2="195.58" width="0.1524" layer="91"/>
+<wire x1="33.02" y1="195.58" x2="33.02" y2="200.66" width="0.1524" layer="91"/>
+<pinref part="U$7" gate="G$2" pin="5"/>
+<wire x1="22.86" y1="198.12" x2="22.86" y2="195.58" width="0.1524" layer="91"/>
+<junction x="22.86" y="195.58"/>
+</segment>
+</net>

Commit message: latest
Parts:
- removed C20, C21: 0.1uF, rcl:C-EUC1206
- removed DSR1: 150, rcl:R-US_R1206
- removed DSR2: 500, rcl:R-US_R1206
- removed DSR3: 1K, rcl:R-US_R1206
- removed IC3: MAX6520, maxim:MAX6520
- removed JP1: gauge_selector, pinhead:PINHD-1X3
- removed RSNS: (no value), rcl:R-US_R1206
- removed U$1: DS2781E, fuelgauge:DS2781E
- removed U$5: JST-PH_2-PIN_HEADER, SRG:JST-PH_2-PIN_HEADER
- removed ZD1: 5.6V, diode:ZENER-DIODESOD80C
- MAX_C1, MAX_C2: device adafruit:CPOL-USD/7343-31W -> rcl:CPOL-USCT7343
Connections:
- removed net BATT-: C20.2, C21.2, IC3.GND, RSNS.2, U$1.VSS, U$5.2
- removed net FG2_VCC: JP1.1, JP12.3
- removed net N$31: DSR1.2, U$1.DQ, ZD1.C
- removed net N$36: C21.1, DSR2.1, U$1.VDD
- removed net N$37: C20.1, U$1.OVD, U$1.VB
- removed net N$39: DSR3.1, U$1.VIN
- removed net REAL_BATT+: DSR2.2, DSR3.2, JP1.3, U$5.1
- net BATT+: now also JP12.3; no longer JP1.2
- net DS_DATA: no longer DSR1.1
- net GND: no longer IC3.IN, IC3.OUT, RSNS.1, U$1.SNS, ZD1.A
- net PIO: no longer U$1.PIO
